File: examples/planar-flyback-5w/kicad/PS-FLYBACK-5W.kicad_pcb (KiCad board)
At the start: 6 copper layers, 50 x 104 mm, 29 parts, among them J1 18-36 V DC, J2 5 V / 1 A isolated, T1 PLANAR 4:2 / Lm 12uH, U1 LT8302ES8E#PBF

Commit message: Replace flyback fuse and correct sourcing scope and 3D model
Parts:
- F1: value 1 A / 63 V fast -> 1 A / 63 V DC fast; footprint Flyback:Fuse_1206_3216Metric -> Flyback:Fuse_Bourns_SF1206F

Commit message: Improve flyback feedback-current margin and prototype clamp budget
Parts:
- R3: value 106k 0.1% -> 115k 0.1%
- R4: value 10k 0.1% -> 10.8k 0.1%
- R5: value 118k 1% -> 128k 0.1%

Commit message: Prepare stocked flyback BOM and JLCPCB assembly review panel
Parts:
- C6: value 470p / 450 V C0G -> 470p / 100 V C0G
- R3: value 115k 0.1% -> 113k 0.1%
- R4: value 10.8k 0.1% -> 10.7k 0.1%
- R5: value 128k 0.1% -> 127k 0.1%
- R6: value 39R 0.66 W -> 39R 0.75 W
- R8: value 2.2R 1.5 W -> 2.2R 2 W; footprint Flyback:R_2512_6332Metric -> Flyback:R_Bourns_CRM2512
- U1: value LT8302ES8E#PBF -> LT8302IS8E#PBF
