File: examples/planar-flyback-5w/kicad/PS-FLYBACK-5W.kicad_sch (KiCad schematic)
At the start: 29 parts, among them J1 18-36 V DC, J2 5 V / 1 A isolated, T1 PLANAR 4:2 / Lm 12uH, U1 LT8302ES8E#PBF

Commit message: Improve flyback feedback-current margin and prototype clamp budget
Parts:
- R3: value 106k 0.1% -> 115k 0.1%; LCSC C4185599 -> (none); MPN TNPW0603106KBEEN -> TNPW0603115KBEEA
- R4: value 10k 0.1% -> 10.8k 0.1%; LCSC C95204 -> (none); MPN RT0603BRD0710KL -> TNPW060310K8BEEA; Manufacturer Yageo -> Vishay
- R5: value 118k 1% -> 128k 0.1%; LCSC C137804 -> (none); MPN RC0603FR-07118KL -> TNPW0603128KBEEA; Manufacturer Yageo -> Vishay
Other:
- note added: "Tune clamp/snubber: SW-VIN peak <=17.5 V, including overshoot."
- note removed: "Tune the clamp and snubber against measured switch overshoot."

Commit message: Prepare stocked flyback BOM and JLCPCB assembly review panel
Parts:
- C5: LCSC C377756 -> C77045; MPN CL10A475KO8NQNC -> GRM188R61C475KE11D; Manufacturer Samsung Electro-Mechanics -> Murata
- C6: value 470p / 450 V C0G -> 470p / 100 V C0G; LCSC C2172062 -> C513677; MPN CGA4C4C0G2W471J060AA -> CC0805JRNPO0BN471; Manufacturer TDK -> Yageo
- R3: value 115k 0.1% -> 113k 0.1%; LCSC (none) -> C705718; MPN TNPW0603115KBEEA -> RT0603BRD07113KL; Manufacturer Vishay -> Yageo
- R4: value 10.8k 0.1% -> 10.7k 0.1%; LCSC (none) -> C861078; MPN TNPW060310K8BEEA -> RT0603BRD0710K7L; Manufacturer Vishay -> Yageo
- R5: value 128k 0.1% -> 127k 0.1%; LCSC (none) -> C705722; MPN TNPW0603128KBEEA -> RT0603BRD07127KL; Manufacturer Vishay -> Yageo
- R6: value 39R 0.66 W -> 39R 0.75 W; LCSC C4059605 -> C6683830; MPN ERJ-P08F39R0V -> SR1206FR-7T39RL; Manufacturer Panasonic -> Yageo
- R8: value 2.2R 1.5 W -> 2.2R 2 W; footprint Flyback:R_2512_6332Metric -> Flyback:R_Bourns_CRM2512; LCSC C4168885 -> C840598; MPN CRCW25122R20FKEGHP -> CRM2512-JW-2R2ELF; Manufacturer Vishay -> Bourns
- U1: value LT8302ES8E#PBF -> LT8302IS8E#PBF; LCSC C117331 -> C673679; MPN LT8302ES8E#PBF -> LT8302IS8E#PBF
