File: examples/planar-gan-60w/kicad/PS-GAN-60W.kicad_sch (KiCad schematic)
At the start: 82 parts, among them J1 XT30 48V INPUT, J2 XT30 12V OUTPUT, Q1 CSD18543Q3A, Q2 CSD18543Q3A, T1 4:2:2 / Lm 13.12uH, U1 LMG2100R044RARR, U2 UCC25600DR, U3 UCC24624DR, U4 LM5164DDAR, U5 TPS7A2450DBVR, U6 EL357N(A)(TA)-VG, U7 TL431AIDBZR, U8 EL357N(A)(TA)-VG, U9 TL431AIDBZR

Commit message: Redraw GaN schematic and compact the bench-accessible A2 board
Parts:
- C7, C8: value 100nF/100V C0G -> 100nF/100V
- D2: value BAT54SLT1G -> BAT54S
- J1: value XT30 48V INPUT -> 48 V INPUT; footprint PS:AMASS_XT30PW-M_1x02_P2.50mm_Horizontal -> PS:CONN-TH_2P-P5.08_WJ2EDGRC-5.08-2P; Design_note AMASS XT30PW-M30.G.Y; pin 2 positive, pin 1 return; through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 -> 5.08 mm pluggable terminal header; pin 2 positive, pin 1 re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; LCSC C431092 -> C3697; MPN XT30PW-M30.G.Y -> WJ2EDGRC-5.08-02P-14-00A; Manufacturer Changzhou Amass Elec -> Ningbo Kangnex Elec
- J2: value XT30 12V OUTPUT -> 12 V / 5 A; footprint PS:AMASS_XT30PW-F_1x02_P2.50mm_Horizontal -> PS:CONN-TH_2P-P5.08_WJ2EDGRC-5.08-2P; Design_note AMASS XT30PW-F20.G.Y; pin 2 positive, pin 1 return; through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 -> 5.08 mm pluggable terminal header; pin 2 positive, pin 1 re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; LCSC C2913282 -> C3697; MPN XT30PW-F20.G.Y -> WJ2EDGRC-5.08-02P-14-00A; Manufacturer Changzhou Amass Elec -> Ningbo Kangnex Elec
- T1: value 4:2:2 / Lm 13.12uH -> 4 : 2 : 2 / ELP22
- U1: value LMG2100R044RARR -> LMG2100R044
- U2: value UCC25600DR -> UCC25600
- U3: value UCC24624DR -> UCC24624
- U4: value LM5164DDAR -> LM5164
- U5: value TPS7A2450DBVR -> TPS7A2450
- U6, U8: value EL357N(A)(TA)-VG -> EL357N
- U7, U9: value TL431AIDBZR -> TL431A
Connections:
- no-connect marks 10 -> 1
Other:
- note added: "01 PLANAR POWER PATH"
- note added: "02 FREQUENCY CONTROL"
- note added: "03 LOCAL BIAS · 48 V → 12 V BUCK → 5 V LOGIC"
- note added: "04 ISOLATED VOLTAGE FEEDBACK · NOMINAL 12.05 V"
- note added: "05 INDEPENDENT OUTPUT OVERVOLTAGE · NOMINAL 13.27 V"
- note added: "48 V nominal → isolated 12 V / 5 A target | A2 engineering prototype"
- note added: "AGND joins PGND inside U1 only."
- note added: "Functional isolation only."
- note added: "PRIMARY"
- note added: "PS-GAN-60W"
- note added: "Primary midpoint is internal copper."
- note added: "R4/R5 and R6/R7: 12 V drive → ~3.7 V logic"
- note added: "SECONDARY"
- note added: "UNBUILT · Functional isolation only · Verify magnetics, switching, no-load operation and thermal limits before release."
- note removed: "01 INPUT / GaN HALF BRIDGE / PLANAR LLC TANK"
- note removed: "02 SYNCHRONOUS RECTIFICATION / ISOLATED OUTPUT"
- note removed: "03 FREQUENCY CONTROL / SIGNAL LEVELS / CURRENT LIMIT"
- note removed: "04 ISOLATED FEEDBACK / OUTPUT OVERVOLTAGE"
- note removed: "05 LOCAL 12 V AND 5 V BIAS — TI LM5164 REFERENCE NETWORK"
- note removed: "12.05 V nominal feedback; 13.27 V nominal OVP. Compensation and light-load behavior require bench tuning."
- note removed: "48 V to isolated 12 V / 5 A • Revision A1 engineering prototype • 2026-10-10"
- note removed: "8 layers / 70 um copper requested. Functional isolation only; no certified safety barrier."
- note removed: "Cr = C7 + C8 = 200 nF; fr ≈ 193 kHz including 0.1 uH leakage allowance."
- note removed: "PS–GaN–60W"
- note removed: "Primary series midpoint (pin 6) is internal winding copper; no external connection."
- note removed: "R4/R5 and R6/R7 translate 12 V GD outputs to 3.7 V logic. Do not bypass."
- note removed: "REVIEW ONLY — NOT RELEASED FOR FABRICATION. See project review for sourcing, electrical assumptions and validation status."
- note removed: "T1: two 0.05 mm gapped ELP22 N87 halves; four primary turns, two per half-secondary."
- company: Planar Studio / KiStack workflow -> Planar Studio
- title: PS-GAN-60W: planar LLC engineering prototype -> PS-GAN-60W: planar LLC converter
- moved on the sheet: C1, C10, C11, C12, C13, C14, C15, C16, C17, C18, C19, C2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

Commit message: Improve GaN example schematic spacing and readability
Parts:
- C1, C19, C2: value 2.2uF/100V -> 2.2uF; Voltage (none) -> 100V
- C10, C12, C25, C5: value 1uF/25V -> 1uF; Voltage (none) -> 25V
- C11, C26: value 2.2uF/25V -> 2.2uF; Voltage (none) -> 25V
- C13, C14, C15, C16, C21, C22: value 22uF/25V -> 22uF; Voltage (none) -> 25V
- C17, C18, C27, C29: value 10nF/50V -> 10nF; Voltage (none) -> 50V
- C20: value 2.2nF/50V -> 2.2nF; Voltage (none) -> 50V
- C23: value 3.3nF/50V -> 3.3nF; Voltage (none) -> 50V
- C24: value 56pF/50V -> 56pF; Voltage (none) -> 50V
- C28: value 1nF/50V -> 1nF; Voltage (none) -> 50V
- C3: value 100nF/100V C0G -> 100nF; Voltage (none) -> 100V C0G
- C4, C6, C9: value 100nF/50V -> 100nF; Voltage (none) -> 50V
- C7, C8: value 100nF/100V -> 100nF; Voltage (none) -> 100V
Connections:
- net BIAS_BST: no longer names the net of C20.1, U4.7 (BST)
- net BIAS_EN: no longer names the net of R14.2, R15.1, U4.3 (EN/UVLO)
- net COMP: no longer names the net of C27.1, R24.2
- net CS_AC: no longer names the net of C17.2, R8.1
- net CS_RECT: no longer names the net of D2.3 (A/C), R8.2
- net DT: no longer names the net of R1.1, U2.1 (DT)
- net FB_K: no longer names the net of C28.1, R21.2, R24.1, U6.2 (CA), U7.1 (CATHODE)
- net FB_LED: no longer names the net of R20.2, R21.1, U6.1 (AN)
- net GD1: no longer names the net of R4.1, U2.8 (GD1)
- net GD2: no longer names the net of R6.1, U2.5 (GD2)
- net HB: no longer names the net of C4.1, U1.10 (HB)
- net OV_K: no longer names the net of R26.2, U8.2 (CA), U9.1 (CATHODE)
- net OV_LED: no longer names the net of R25.2, R26.1, U8.1 (AN)
- net OV_REF: no longer names the net of C29.1, R27.2, R28.1, U9.2 (REF)
- net PRI_A: no longer names the net of L1.2, T1.1 (P_DOT)
- net RIPPLE: no longer names the net of C23.1, C24.1, R19.2
- net RON: no longer names the net of R16.2, U4.4 (RON)
- net RT: no longer names the net of R2.1, R3.1, U2.2 (RT)
- net SR_G1: no longer names the net of Q1.4 (G), R10.2
- net SR_G2: no longer names the net of Q2.4 (G), R11.2
- net SR_REG: no longer names the net of C11.1, U3.3 (REG)
- net VG1: no longer names the net of R10.1, U3.1 (VG1)
- net VG2: no longer names the net of R11.1, U3.8 (VG2)
- net VREF: no longer names the net of C27.2, C28.2, R22.2, R23.1, U7.2 (REF)
- net VS1: no longer names the net of R12.2, U3.4 (VD1)
- net VS2: no longer names the net of R13.2, U3.6 (VD2)
Other:
- note added: "48 V nominal → isolated 12 V / 5 A target | A3 schematic · A2 hardware"
- note added: "PGND: input return / SGND: isolated output return / AGND: controller return (joins PGND inside U1)"
- note removed: "48 V nominal → isolated 12 V / 5 A target | A2 engineering prototype"
- note removed: "PRIMARY"
- note removed: "SECONDARY"
- moved on the sheet: C17, C24, R10, R11, R12, R13, R8

Commit message: Wire sense and bias circuits cohesively in GaN schematic
Connections:
- net BIAS_FB: no longer names the net of C24.2, R17.2, R18.1, U4.5 (FB)
- net BIAS_SW: no longer names the net of C20.2, L2.1, R19.1, U4.8 (SW)
- net OC: no longer names the net of C18.1, D2.2 (C), R9.1, U2.3 (OC)
- net SEC_A: no longer names the net of Q1.5 (D), Q1.6 (D), Q1.7 (D), Q1.8 (D), Q1.9 (D), R12.1, T1.3 (S_DOT)
- net SEC_B: no longer names the net of Q2.5 (D), Q2.6 (D), Q2.7 (D), Q2.8 (D), Q2.9 (D), R13.1, T1.5 (S_END)
Other:
- note added: "03 LOCAL BIAS · 12 V + 5 V"
- note added: "04 ISOLATED FEEDBACK · 12.05 V"
- note added: "05 OUTPUT OV PROTECTION · 13.27 V"
- note added: "12 V drive → ~3.7 V logic"
- note added: "48 V nominal → isolated 12 V / 5 A target | A4 schematic · A2 hardware"
- note removed: "03 LOCAL BIAS · 48 V → 12 V BUCK → 5 V LOGIC"
- note removed: "04 ISOLATED VOLTAGE FEEDBACK · NOMINAL 12.05 V"
- note removed: "05 INDEPENDENT OUTPUT OVERVOLTAGE · NOMINAL 13.27 V"
- note removed: "48 V nominal → isolated 12 V / 5 A target | A3 schematic · A2 hardware"
- note removed: "AGND joins PGND inside U1 only."
- note removed: "R4/R5 and R6/R7: 12 V drive → ~3.7 V logic"
- moved on the sheet: C10, C17, C18, C20, C21, C22, C23, C24, C25, C26, C9, D2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

Commit message: Clarify GaN schematic and correct LM5164 RON grounding
Parts:
- R16: Design_note (none) -> 100k RON timing resistor to PGND per TI LM5164 Rev D pin 4 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
Connections:
- net PGND: now also R16.1
- net VIN: no longer R16.1
Other:
- note added: "48 V nominal → isolated 12 V / 5 A target | A5 schematic · A3 hardware"
- note removed: "48 V nominal → isolated 12 V / 5 A target | A4 schematic · A2 hardware"
- moved on the sheet: C1, C11, C2, C3, F1, J1, J2, R12, R14, R15, R16, TP1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

Commit message: Tighten GaN switching loops and separate rectifier sense return
Parts:
- U1: Design_note (none) -> HS is internally connected to SW. Dedicated local C4 return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
Connections:
- net SW: no longer C4.2, U1.11 (HS)
- new net: C4.2, U1.11 (HS)
Other:
- note added: "48 V nominal → isolated 12 V / 5 A target | A6 schematic · A4 hardware"
- note removed: "48 V nominal → isolated 12 V / 5 A target | A5 schematic · A3 hardware"

Commit message: Refine GaN example return paths and rectifier placement
Parts:
- C10: footprint PS:C_0603_1608Metric -> PS:C_0805_2012Metric; Design_note (none) -> UCC25600 Rev D sections 9-10: 1 uF, 0805, 50 V X7R directly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; LCSC C86020 -> C28323; MPN GRM188R71E105KA12D -> CL21B105KBFNNNE; Manufacturer Murata Electronics -> Samsung Electro-Mechanics; Voltage 25V -> 50V
Other:
- note added: "48 V nominal → isolated 12 V / 5 A target | A7 schematic · A5 hardware"
- note removed: "48 V nominal → isolated 12 V / 5 A target | A6 schematic · A4 hardware"

Commit message: Refine GaN layout and add verified ground stitching
Other:
- note added: "48 V nominal → isolated 12 V / 5 A target | A8 schematic · A6 hardware"
- note removed: "48 V nominal → isolated 12 V / 5 A target | A7 schematic · A5 hardware"

Commit message: Improve GaN bias routing and audit component stress ratings
Parts:
- C17: Design_note (none) -> 100 V AC-coupling capacitor. Steady DC is about VIN/2; rais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; LCSC C100042 -> C107059; MPN CC0603KRX7R9BB103 -> CC0603KRX7R0BB103; Voltage 50V -> 100V
- F1: value 2A / 63V -> 3A / 65V; Design_note Fuse does not guarantee semiconductor protection -> 3 A / 65 V fuse selected for operating-current temperature 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; LCSC C719183 -> C3177336; MPN SF-1206F200-2 -> SF-1206F300M-2
- R20, R25: Design_note (none) -> High-power 0603. Use conservative catalog rating 0.25 W at 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; LCSC C114668 -> C543357; MPN RC0603FR-071K5L -> ERJPA3F1501V; Manufacturer YAGEO -> Panasonic
- R8: value 15kR -> 24.9kR; Design_note (none) -> Revised from 15k to avoid predicted full-load nuisance OC t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; LCSC C114661 -> C137761; MPN RC0603FR-0715KL -> RC0603FR-0724K9L
Other:
- note added: "48 V nominal → isolated 12 V / 5 A target | A9 schematic · A7 hardware"
- note removed: "48 V nominal → isolated 12 V / 5 A target | A8 schematic · A6 hardware"
