File: examples/planar-gan-60w/kicad/PS-GAN-60W.kicad_sch (KiCad schematic)
At the start: 82 parts, among them J1 48 V INPUT, J2 12 V / 5 A, Q1 CSD18543Q3A, Q2 CSD18543Q3A, T1 4 : 2 : 2 / ELP22, U1 LMG2100R044, U2 UCC25600, U3 UCC24624, U4 LM5164, U5 TPS7A2450, U6 EL357N, U7 TL431A, U8 EL357N, U9 TL431A

Commit message: Improve GaN reference planes and output distribution from layout review
Other:
- note added: "48 V nominal → isolated 12 V / 5 A target | A10 schematic · A8 hardware"
- note removed: "48 V nominal → isolated 12 V / 5 A target | A9 schematic · A7 hardware"

Commit message: Repair GaN manufacturing geometry and purposeful copper pours (A11)
Other:
- note added: "48 V nominal → isolated 12 V / 5 A target | A11 engineering prototype"
- note removed: "48 V nominal → isolated 12 V / 5 A target | A10 schematic · A8 hardware"

Commit message: Clean GaN routing and silkscreen; supply single-board A12 files
Other:
- note added: "48 V nominal → isolated 12 V / 5 A target | A12 engineering prototype"
- note removed: "48 V nominal → isolated 12 V / 5 A target | A11 engineering prototype"
