File: examples/coil-tile/kicad/CoilTile.kicad_pcb (KiCad board)
At the start: 4 copper layers, 72 x 90 mm, 32 parts, among them J1 USB-C / USB 2.0, U1 AP2112K-3.3TRG1, U2 MCP2221A-I/ST, U3 LDC1614RGHR, U4 USBLC6-2SC6

Commit message: Refine CoilTile A3 schematic and PCB routing
Compact the continuous schematic, group unused bridge pins, and clarify service notes.
Shorten SDA/SCL and CC1 routes, remove the SCL power-plane detour, label service pads,
and move the sensor bypass capacitor closer to VDD.

Preserve electrical nets, pin identities, coil artwork and example mounting holes.
Regenerate checked fabrication files and reviewed previews; record route metrics.
Native ERC, DRC, connectivity and schematic parity pass with zero issues.
Parts:
- moved TP4 16.6 mm to (89.0, 123.0)
- moved TP3 7.81 mm to (81.0, 123.0)
- moved C5 1.50 mm to (88.2, 92.5)
Routing:
- net /SCL: track 82.3 -> 53.1 mm
- net /SDA: track 78.9 -> 62.6 mm
- net /CC1: track 21.7 -> 11.1 mm
- net +3V3: track 19.9 -> 18.1 mm
Other:
- board text added: "A3"
- board text added: "SCL"
- board text added: "SDA"
- board text removed: "A2"
