File: examples/coil-tile/kicad/CoilTile.kicad_sch (KiCad schematic)
At the start: 32 parts, among them J1 USB-C / USB 2.0, U1 AP2112K-3.3TRG1, U2 MCP2221A-I/ST, U3 LDC1614RGHR, U4 USBLC6-2SC6

Commit message: Refine CoilTile A3 schematic and PCB routing
Compact the continuous schematic, group unused bridge pins, and clarify service notes.
Shorten SDA/SCL and CC1 routes, remove the SCL power-plane detour, label service pads,
and move the sensor bypass capacitor closer to VDD.

Preserve electrical nets, pin identities, coil artwork and example mounting holes.
Regenerate checked fabrication files and reviewed previews; record route metrics.
Native ERC, DRC, connectivity and schematic parity pass with zero issues.
Other:
- note added: "01 USB + PROTECTION"
- note added: "02 HID / I2C BRIDGE"
- note added: "03 INDUCTANCE CONVERTER"
- note added: "04 LC SENSORS"
- note added: "0x2A / internal clock / always enabled"
- note added: "24 mm / 16 turns / 0.20 mm trace + gap / 220 pF C0G"
- note added: "5.51 uH and ~4.57 MHz nominal; nearby metal changes L and Q."
- note added: "A3 prototype | 2 x 2 printed coils | USB powered | No firmware programming"
- note added: "BUILD + SERVICE"
- note added: "M3 exposed-substrate edge holes / American Embedded"
- note added: "MCP2221A: VDD and VUSB both supplied from external 3.3 V."
- note added: "SENSOR NOTES"
- note added: "Same mounting geometry as flyback + GaN examples. Use nylon hardware."
- note added: "TP1: 3V3 TP2: GND TP3: SDA TP4: SCL"
- note added: "USB-C: 5 V sink; independent 5.1k CC pull-downs."
- note added: "Unbuilt A3: characterize amplitude, noise and coil coupling."
- note removed: "0x2A / internal clock"
- note removed: "24 mm / 16 turns / 0.20 mm trace + gap"
- note removed: "5 V sink / independent CC pull-downs"
- note removed: "5.51 uH + 220 pF: ~4.57 MHz nominal"
- note removed: "A2 prototype | One continuous signal path | 2 x 2 printed coils | No firmware programming"
- note removed: "Characterize amplitude, noise and coil coupling before reordering."
- note removed: "M3 exposed-substrate edge holes / American Embedded footprint"
- note removed: "Same geometry as the flyback and GaN examples. Use nylon hardware."
- note removed: "UNBUILT A2 PROTOTYPE"
- note removed: "USB-C > HID / I2C BRIDGE > FOUR-CHANNEL SENSOR > LC TANKS"
- note removed: "VDD and VUSB both use external 3.3 V"
- moved on the sheet: C1, C10, C2, C3, C4, C5, C6, C7, C8, C9, H1, H2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
